File: 1_1.kicad_sch (KiCad schematic)
At the start: 36 parts, among them U1 CH32V203C8U6, U18 KH-TYPE-C-16P, U2 HX_PZ2_54-3X2P_ZZ, U26 DMG2305UX-7, U28 DMG2305UX-7, U3 32.768kHz, U5 SD101CWS, X1 8MHz

Commit message: chore: reset components anotation
Parts:
- renumbered C11 to C10, C13 to C11, C6 to C5, C7 to C6, C8 to C7, C9 to C8, C10 to C9, R5 to R3, R7 to R4, R8 to R5, R9 to R6, U18 to U4, U26 to U6, U28 to U7
Changed lines of the file:
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@@
 		(dnp no)
 		(fields_autoplaced yes)
-		(property "Reference" "U18"
+		(property "Reference" "U4"
 			(at 295.91 31.75 0)
 			(effects
@@
 			(project "ch32v203_dev"
 				(path "/0e6f0aa4-a0ff-4959-b558-a36c5faa29c6/695d48d0-b127-49b4-b19c-0382de2ea4d3"
-					(reference "U18")
+					(reference "U4")
 					(unit 1)
 				)
@@
 		(on_board yes)
 		(dnp no)
-		(property "Reference" "R8"
+		(property "Reference" "R5"
 			(at 116.84 49.276 90)
 			(effects
@@
 			(project ""
 				(path "/0e6f0aa4-a0ff-4959-b558-a36c5faa29c6/695d48d0-b127-49b4-b19c-0382de2ea4d3"
-					(reference "R8")
+					(reference "R5")
 					(unit 1)
 				)
@@
 		(on_board yes)
 		(dnp no)
-		(property "Reference" "R9"
+		(property "Reference" "R6"
 			(at 238.76 52.324 90)
 			(effects
@@
 			(project "ch32v203_dev"
 				(path "/0e6f0aa4-a0ff-4959-b558-a36c5faa29c6/695d48d0-b127-49b4-b19c-0382de2ea4d3"
-					(reference "R9")
+					(reference "R6")
 					(unit 1)
 				)
@@
 		(on_board yes)
 		(dnp no)
-		(property "Reference" "R7"
+		(property "Reference" "R4"
 			(at 106.426 49.53 90)
 			(effects
@@
 			(project ""
 				(path "/0e6f0aa4-a0ff-4959-b558-a36c5faa29c6/695d48d0-b127-49b4-b19c-0382de2ea4d3"
-					(reference "R7")
+					(reference "R4")
 					(unit 1)
 				)
@@
 		(on_board yes)
 		(dnp no)
-		(property "Reference" "C11"
+		(property "Reference" "C10"
 			(at 197.612 101.092 90)
 			(effects
@@
 			(project ""
 				(path "/0e6f0aa4-a0ff-4959-b558-a36c5faa29c6/695d48d0-b127-49b4-b19c-0382de2ea4d3"
-					(reference "C11")
+					(reference "C10")
 					(unit 1)
 				)
@@
 		(on_board yes)
 		(dnp no)
-		(property "Reference" "C10"
+		(property "Reference" "C9"
 			(at 197.104 127.762 90)
 			(effects
@@
 			(project ""
 				(path "/0e6f0aa4-a0ff-4959-b558-a36c5faa29c6/695d48d0-b127-49b4-b19c-0382de2ea4d3"
-					(reference "C10")
+					(reference "C9")
 					(unit 1)
 				)
@@
 		(on_board yes)
 		(dnp no)
-		(property "Reference" "C7"
+		(property "Reference" "C6"
 			(at 342.392 153.162 0)
 			(effects
@@
 			(project "usb_sp"
 				(path "/0e6f0aa4-a0ff-4959-b558-a36c5faa29c6/695d48d0-b127-49b4-b19c-0382de2ea4d3"
-					(reference "C7")
+					(reference "C6")
 					(unit 1)
 				)
@@
 		(dnp no)
 		(fields_autoplaced yes)
-		(property "Reference" "U28"
+		(property "Reference" "U7"
 			(at 387.35 116.8399 0)
 			(effects
@@
 			(project "ch32v203_dev"
 				(path "/0e6f0aa4-a0ff-4959-b558-a36c5faa29c6/695d48d0-b127-49b4-b19c-0382de2ea4d3"
-					(reference "U28")
+					(reference "U7")
 					(unit 1)
 				)
@@
 		(on_board yes)
 		(dnp no)
-		(property "Reference" "C6"
+		(property "Reference" "C5"
 			(at 314.706 153.162 0)
 			(effects
@@
 			(project "usb_sp"
 				(path "/0e6f0aa4-a0ff-4959-b558-a36c5faa29c6/695d48d0-b127-49b4-b19c-0382de2ea4d3"
-					(reference "C6")
+					(reference "C5")
 					(unit 1)
 				)
@@
 		(on_board yes)
 		(dnp no)
-		(property "Reference" "R5"
+		(property "Reference" "R3"
 			(at 73.406 46.228 0)
 			(effects
@@
 			(project ""
 				(path "/0e6f0aa4-a0ff-4959-b558-a36c5faa29c6/695d48d0-b127-49b4-b19c-0382de2ea4d3"
-					(reference "R5")
+					(reference "R3")
 					(unit 1)
 				)
@@
 		(dnp no)
 		(fields_autoplaced yes)
-		(property "Reference" "U26"
+		(property "Reference" "U6"
 			(at 314.96 115.5699 0)
 			(effects
@@
 			(project "ch32v203_dev"
 				(path "/0e6f0aa4-a0ff-4959-b558-a36c5faa29c6/695d48d0-b127-49b4-b19c-0382de2ea4d3"
-					(reference "U26")
+					(reference "U6")
 					(unit 1)
 				)
@@
 		(on_board yes)
 		(dnp no)
-		(property "Reference" "C8"
+		(property "Reference" "C7"
 			(at 356.362 153.162 0)
 			(effects
@@
 			(project "usb_sp"
 				(path "/0e6f0aa4-a0ff-4959-b558-a36c5faa29c6/695d48d0-b127-49b4-b19c-0382de2ea4d3"
-					(reference "C8")
+					(reference "C7")
 					(unit 1)
 				)
@@
 		(on_board yes)
 		(dnp no)
-		(property "Reference" "C9"
+		(property "Reference" "C8"
 			(at 330.2 152.908 0)
 			(effects
@@
 			(project "usb_sp"
 				(path "/0e6f0aa4-a0ff-4959-b558-a36c5faa29c6/695d48d0-b127-49b4-b19c-0382de2ea4d3"
-					(reference "C9")
+					(reference "C8")
 					(unit 1)
 				)
@@
 		(on_board yes)
 		(dnp no)
-		(property "Reference" "C13"
+		(property "Reference" "C11"
 			(at 302.768 164.592 90)
 			(effects
@@
 			(project "usb_sp"
 				(path "/0e6f0aa4-a0ff-4959-b558-a36c5faa29c6/695d48d0-b127-49b4-b19c-0382de2ea4d3"
-					(reference "C13")
+					(reference "C11")
 					(unit 1)
 				)
