File: ch32v203_dev.kicad_pcb (KiCad board)
At the start: 4 copper layers, 27.7 x 59.7 mm, 36 parts, among them U1 CH32V203C8U6, U18 KH-TYPE-C-16P, U2 HX_PZ2_54-3X2P_ZZ, U26 DMG2305UX-7, U28 DMG2305UX-7, U3 32.768kHz, U5 SD101CWS, X1 8MHz

Commit message: chore: reset components anotation
Parts:
- renumbered C11 to C10, C13 to C11, C6 to C5, C7 to C6, C8 to C7, C9 to C8, C10 to C9, R5 to R3, R7 to R4, R8 to R5, R9 to R6, U18 to U4, U26 to U6, U28 to U7
Changed lines of the file:
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@@
 	(net 55 "/CH32V203/USB_CC1")
 	(net 56 "/CH32V203/USB_CC2")
-	(net 57 "unconnected-(U18-SUB2-PadB8)")
-	(net 58 "unconnected-(U18-SUB1-PadA8)")
+	(net 57 "unconnected-(U4-SUB2-PadB8)")
+	(net 58 "unconnected-(U4-SUB1-PadA8)")
 	(footprint "Capacitor_SMD:C_0402_1005Metric"
 		(layer "F.Cu")
@@
 		(descr "Capacitor SMD 0402 (1005 Metric), square (rectangular) end terminal, IPC-7351 nominal, (Body size source: IPC-SM-782 page 76, https://www.pcb-3d.com/wordpress/wp-content/uploads/ipc-sm-782a_amendment_1_and_2.pdf), generated with kicad-footprint-generator")
 		(tags "capacitor")
-		(property "Reference" "C7"
+		(property "Reference" "C6"
 			(at 0 -1.16 90)
 			(layer "F.SilkS")
@@
 		(descr "Resistor SMD 0603 (1608 Metric), square (rectangular) end terminal, IPC-7351 nominal, (Body size source: IPC-SM-782 page 72, https://www.pcb-3d.com/wordpress/wp-content/uploads/ipc-sm-782a_amendment_1_and_2.pdf), generated with kicad-footprint-generator")
 		(tags "resistor")
-		(property "Reference" "R9"
+		(property "Reference" "R6"
 			(at 0 -1.43 90)
 			(layer "F.SilkS")
@@
 		(descr "Resistor SMD 0603 (1608 Metric), square (rectangular) end terminal, IPC-7351 nominal, (Body size source: IPC-SM-782 page 72, https://www.pcb-3d.com/wordpress/wp-content/uploads/ipc-sm-782a_amendment_1_and_2.pdf), generated with kicad-footprint-generator")
 		(tags "resistor")
-		(property "Reference" "R5"
+		(property "Reference" "R3"
 			(at 3.3528 0 90)
 			(layer "F.SilkS")
@@
 		(descr "Resistor SMD 0402 (1005 Metric), square (rectangular) end terminal, IPC-7351 nominal, (Body size source: IPC-SM-782 page 72, https://www.pcb-3d.com/wordpress/wp-content/uploads/ipc-sm-782a_amendment_1_and_2.pdf), generated with kicad-footprint-generator")
 		(tags "resistor")
-		(property "Reference" "R7"
+		(property "Reference" "R4"
 			(at 0.0298 -1.1392 90)
 			(layer "F.SilkS")
@@
 		(descr "SOT-23-3_L2.9-W1.3-P1.90-LS2.4-BR footprint")
 		(tags "SOT-23-3_L2.9-W1.3-P1.90-LS2.4-BR footprint C150470")
-		(property "Reference" "U28"
+		(property "Reference" "U7"
 			(at 0 -3.526213 90)
 			(layer "F.SilkS")
@@
 		(descr "Resistor SMD 0402 (1005 Metric), square (rectangular) end terminal, IPC-7351 nominal, (Body size source: IPC-SM-782 page 72, https://www.pcb-3d.com/wordpress/wp-content/uploads/ipc-sm-782a_amendment_1_and_2.pdf), generated with kicad-footprint-generator")
 		(tags "resistor")
-		(property "Reference" "R8"
+		(property "Reference" "R5"
 			(at 1.29 0.9 0)
 			(layer "F.SilkS")
@@
 		(descr "Capacitor SMD 0402 (1005 Metric), square (rectangular) end terminal, IPC-7351 nominal, (Body size source: IPC-SM-782 page 76, https://www.pcb-3d.com/wordpress/wp-content/uploads/ipc-sm-782a_amendment_1_and_2.pdf), generated with kicad-footprint-generator")
 		(tags "capacitor")
-		(property "Reference" "C10"
+		(property "Reference" "C9"
 			(at 2.411 -0.234 0)
 			(layer "F.SilkS")
@@
 		(descr "Capacitor SMD 0402 (1005 Metric), square (rectangular) end terminal, IPC-7351 nominal, (Body size source: IPC-SM-782 page 76, https://www.pcb-3d.com/wordpress/wp-content/uploads/ipc-sm-782a_amendment_1_and_2.pdf), generated with kicad-footprint-generator")
 		(tags "capacitor")
-		(property "Reference" "C13"
+		(property "Reference" "C11"
 			(at 0 -1.16 0)
 			(layer "F.SilkS")
@@
 		(descr "Capacitor SMD 0402 (1005 Metric), square (rectangular) end terminal, IPC-7351 nominal, (Body size source: IPC-SM-782 page 76, https://www.pcb-3d.com/wordpress/wp-content/uploads/ipc-sm-782a_amendment_1_and_2.pdf), generated with kicad-footprint-generator")
 		(tags "capacitor")
-		(property "Reference" "C6"
+		(property "Reference" "C5"
 			(at 0 -1.16 180)
 			(layer "F.SilkS")
@@
 		(descr "USB-C-SMD_KH-TYPE-C-16P footprint")
 		(tags "USB-C-SMD_KH-TYPE-C-16P footprint C709357")
-		(property "Reference" "U18"
+		(property "Reference" "U4"
 			(at -0.000025 -4.415037 0)
 			(layer "F.SilkS")
@@
 			(size 0.3 1.3)
 			(layers "F.Cu" "F.Mask" "F.Paste")
-			(net 58 "unconnected-(U18-SUB1-PadA8)")
+			(net 58 "unconnected-(U4-SUB1-PadA8)")
 			(pinfunction "SUB1")
 			(pintype "unspecified")
@@
 			(size 0.3 1.3)
 			(layers "F.Cu" "F.Mask" "F.Paste")
-			(net 57 "unconnected-(U18-SUB2-PadB8)")
+			(net 57 "unconnected-(U4-SUB2-PadB8)")
 			(pinfunction "SUB2")
 			(pintype "unspecified")
@@
 		(descr "Capacitor SMD 0402 (1005 Metric), square (rectangular) end terminal, IPC-7351 nominal, (Body size source: IPC-SM-782 page 76, https://www.pcb-3d.com/wordpress/wp-content/uploads/ipc-sm-782a_amendment_1_and_2.pdf), generated with kicad-footprint-generator")
 		(tags "capacitor")
-		(property "Reference" "C9"
+		(property "Reference" "C8"
 			(at 0 -1.16 0)
 			(layer "F.SilkS")
@@
 		(descr "Capacitor SMD 0402 (1005 Metric), square (rectangular) end terminal, IPC-7351 nominal, (Body size source: IPC-SM-782 page 76, https://www.pcb-3d.com/wordpress/wp-content/uploads/ipc-sm-782a_amendment_1_and_2.pdf), generated with kicad-footprint-generator")
 		(tags "capacitor")
-		(property "Reference" "C8"
+		(property "Reference" "C7"
 			(at 0 -1.16 0)
 			(layer "F.SilkS")
@@
 		(descr "SOT-23-3_L2.9-W1.3-P1.90-LS2.4-BR footprint")
 		(tags "SOT-23-3_L2.9-W1.3-P1.90-LS2.4-BR footprint C150470")
-		(property "Reference" "U26"
+		(property "Reference" "U6"
 			(at 0 -3.526213 90)
 			(layer "F.SilkS")
@@
 		(descr "Capacitor SMD 0402 (1005 Metric), square (rectangular) end terminal, IPC-7351 nominal, (Body size source: IPC-SM-782 page 76, https://www.pcb-3d.com/wordpress/wp-content/uploads/ipc-sm-782a_amendment_1_and_2.pdf), generated with kicad-footprint-generator")
 		(tags "capacitor")
-		(property "Reference" "C11"
+		(property "Reference" "C10"
 			(at -0.2012 -1.9619 270)
 			(layer "F.SilkS")
